Commit message: Update explicit parameters into de xacro

File: onrobot_2fg7_gripper_description/robots/2fg7_gripper.urdf.xacro (robot description, xacro)
@@ -5,5 +5,8 @@
 	<xacro:arg name="prefix" default="robot_"/>
 	<xacro:arg name="gripper_prefix" default="$(arg prefix)gripper"/>
-  <xacro:property name="PI" value="3.1415926535897931"/>
+	<xacro:arg name="robot_ip" default="192.168.0.210"/>
+	<xacro:arg name="interpreter_port" default="30020"/>
+	<xacro:arg name="tool_index" default="0"/>
+	  <xacro:property name="PI" value="3.1415926535897931"/>
   <!-- Gripper -->
   <xacro:onrobot_2fg7_gripper prefix="$(arg gripper_prefix)" parent="$(arg prefix)arm_tool0">
@@ -13,4 +16,8 @@
     <hardware>
       <plugin>ur_gripper_controller/URGripperController</plugin>
+      <param name="robot_ip">$(arg robot_ip)</param>
+      <param name="interpreter_port">$(arg interpreter_port)</param>
+      <param name="gripper_plugin">ur_gripper_plugins/OR2FG7Gripper</param>
+      <param name="tool_index">$(arg tool_index)</param>
     </hardware>
     <joint name="$(arg gripper_prefix)_left_finger_joint">
